File: Order339582-10x10-SandyNoble-Polarshieldv1.5.brd (EAGLE design)
At the start: 100 x 80 mm, 62 parts, among them CN1 1X4-CLEANBIG, CN2 1X4-CLEANBIG, J1 1X2-3.5MM, U1 ARDUINO_MEGA_SHIELD, X1 2.1MMJACKTHM

Commit message: Finished v1.5 and sent off to be made.
Parts:
- added R3, R4, R6: 100, rcl:R0805
- added T_STP, X_STP, Y_STP: (no value), led:CHIP-LED0805
- moved RN6 45.9 mm to (34.7, 12.4), turned to 270 degrees
- moved TX_LED 9.16 mm to (27.9, 5.08), turned to 90 degrees
- moved D13 8.07 mm to (27.9, 10.2)
- moved RX_LED 3.59 mm to (27.9, 7.62), turned to 90 degrees
- moved C2 2.62 mm to (17.0, 42.9)
- moved PWR 0.91 mm to (27.9, 2.54), turned to 90 degrees
Connections:
- net T-DIR renamed X-DIR
- net T-EN renamed X-EN
- removed net T-STEP: CN1.4, U$6.STEP, U1.D31
- new net N$23: R3.1, T_STP.A
- new net X-STEP: CN1.4, R3.2, U$6.STEP, U1.D31
- net GND: now also T_STP.C, X_STP.C, Y_STP.C
- net N$15: now also RN6.2, RX_LED.C; no longer TX_LED.C
- net N$16: now also RN6.3, TX_LED.C; no longer RX_LED.C
- net N$18: now also R4.1, Y_STP.A; no longer RN6.3, TX_LED.A
- net N$19: now also R6.1, X_STP.A; no longer RN6.2, RX_LED.A
- net N$2: now also RN6.4; no longer RN6.1
- net VCC: now also RN6.5, RX_LED.A, TX_LED.A; no longer RN6.8
- net Y-STEP: now also R4.2
- net Z-STEP: now also R6.2
Routing:
- net SERV2: track 63.3 -> 243.5 mm, vias 1 -> 15
- net X-STEP: track 0.00 -> 116.8 mm, vias 0 -> 3
- net D1: track 2.59 -> 75.6 mm, vias 0 -> 7
- net T-STEP: track 69.1 -> 0.00 mm
- net D0: track 2.59 -> 58.8 mm, vias 0 -> 3
- net Z-STEP: track 21.4 -> 69.2 mm, vias 0 -> 3
- net N$16: track 0.00 -> 24.0 mm, vias 0 -> 2
- net N$18: track 0.00 -> 19.6 mm, vias 0 -> 2
- net VCC: track 291.5 -> 304.7 mm
- net GND: track 505.8 -> 519.0 mm, vias 5 -> 7
- net LED: track 92.7 -> 80.9 mm, vias 3 -> 6
- net N$15: track 0.00 -> 10.9 mm
- net N$2: track 4.11 -> 14.9 mm, vias 0 -> 2
- net Y-STEP: track 44.7 -> 49.6 mm
- net N$19: track 0.00 -> 3.02 mm
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- added copper zone on layer 1, net GND
- added copper zone on layer 16, net GND
Other:
- board text added: "10K"
- board text added: "2013.09.01 #339582"
- board text removed: "2013.08.28 #339499"
