File: OrderPIEF101613-03_10x10-SandyNoble-Polarshieldv1.6.sch (EAGLE design)
At the start: 60 parts, among them CN1 1X4-CLEANBIG, CN2 1X4-CLEANBIG, J1 1X2-3.5MM, U1 ARDUINO_MEGA_SHIELD, X1 2.1MMJACKTHM

Commit message: Merged a resistor into a network and changed a few values, also cleaned up silkscreen.
Parts:
- removed R41: 1K, rcl:R-EU_R0805
- added R3: 1K, rcl:R-EU_R0805
- added R6: 1k, rcl:R-EU_R0805
- added RN6: 1K, resistor-dil:4R-NEXBS8V
- added RX_LED, TX_LED, T_STP, X_STP, Y_STP: (no value), led:LEDCHIP-LED0805
- R1, R5, R8: value 100k -> 1k
- renumbered POWER to PWR
Connections:
- net T-DIR renamed X-DIR
- net T-EN renamed X-EN
- removed net T-STEP: CN1.4, U$6.STEP, U1.D31
- new net N$15: RN6B.1, RX_LED.C
- new net N$16: RN6C.1, TX_LED.C
- new net N$18: RN6A.1, Y_STP.A
- new net N$19: R6.1, X_STP.A
- new net N$23: R3.1, T_STP.A
- new net X-STEP: CN1.4, R3.2, U$6.STEP, U1.D31
- net D0: now also RN6B.2
- net D1: now also RN6C.2
- net GND: now also T_STP.C, X_STP.C, Y_STP.C
- net N$2: now also RN6D.1; no longer R41.1
- net VCC: now also RN6D.2, RX_LED.A, TX_LED.A; no longer R41.2
- net Y-STEP: now also RN6A.2
- net Z-STEP: now also R6.2
