File: Polarshield v2.0d.brd (EAGLE design)
At the start: 100 x 80 mm, 74 parts, among them IC1 MP2307, IC2 74541PW, IC3 74541PW, IC4 74541PW, IC5 74541PW, J1 1X2-3.5MM, U1 ARDUINO_MEGA_SHIELD, X1 2.1MMJACKTHM

Commit message: v2.0d
Parts:
- moved SER1 2.54 mm to (21.6, 73.7)
- moved SER2 2.54 mm to (21.6, 71.1)
- moved C6 2.41 mm to (23.4, 67.6)
Routing:
- net VCC: track 423.9 -> 428.0 mm
- net +12V: track 164.1 -> 167.0 mm
- net SERV2: track 41.0 -> 38.5 mm
- net N$20: track 18.2 -> 15.9 mm
- net N$15: track 9.94 -> 9.04 mm
- net SERV1: track 39.8 -> 40.6 mm
- net GND: vias 71 -> 74
Other:
- board text added: "Polarshield v2.0d"
- board text added: "Polarshield v2.0d An open source art project. www.polargraph.co.uk 2014.07.30"
- board text added: "Polarshield v2.0d www.polargraph.co.uk 2014.07.30"
- board text removed: "Polarshield v2.0c"
- board text removed: "Polarshield v2.0c An open source art project. www.polargraph.co.uk 2014.06.07"
- board text removed: "Polarshield v2.0c www.polargraph.co.uk 2014.06.07"
