File: Polarshield v2.1.brd (EAGLE design)
At the start: 100 x 80 mm, 82 parts, among them IC1 MP2307, IC2 74541PW, IC3 74541PW, IC4 74541PW, IC5 74541PW, J1 1X2-3.5MM, U1 ARDUINO_MEGA_SHIELD, X1 2.1MMJACKTHM

Commit message: Ran the DRU, ready for making.
Parts:
- removed CN5, CN6: (no value), Polarshield v2.0e:1X04-CLEANBIG
- added JP4, JP5, JP6, JP7: (no value), SparkFun-Connectors:1X02_PP_HOLES_ONLY
- JP1, JP3: device SparkFun-Connectors:1X02_NO_SILK -> SparkFun-Connectors:1X02_PP_HOLES_ONLY
- JP2: device SparkFun-Connectors:1X03_NO_SILK -> SparkFun-Connectors:1X03_PP_HOLES_ONLY
Connections:
- net D42: now also JP4.2; no longer CN5.4
- net D43: now also JP4.1; no longer CN6.4
- net D44: now also JP5.2; no longer CN5.3
- net D45: now also JP5.1; no longer CN6.3
- net D46: now also JP6.2; no longer CN5.2
- net D47: now also JP6.1; no longer CN6.2
- net D48: now also JP7.2; no longer CN5.1
- net D49: now also JP7.1; no longer CN6.1
Routing:
- net RESET: track 105.6 -> 107.6 mm
- net GND: vias 85 -> 84

Commit message: v2.1
Parts:
- removed JP15: (no value), pinhead:2X03
- added X-MAX, X-MIN, Y-MAX, Y-MIN: (no value), ultimachine:3PIN-HEADER
Connections:
- net GND: now also X-MAX.1, X-MIN.1, Y-MAX.1, Y-MIN.1; no longer JP15.6
- net VCC: now also X-MAX.2, X-MIN.2, Y-MAX.2, Y-MIN.2; no longer JP15.5
- net X-MAX: now also X-MAX.3; no longer JP15.3
- net X-MIN: now also X-MIN.3; no longer JP15.1
- net Y-MAX: now also Y-MAX.3; no longer JP15.4
- net Y-MIN: now also Y-MIN.3; no longer JP15.2
Routing:
- net Y-MIN: track 39.8 -> 27.8 mm
- net X-MIN: track 36.9 -> 26.1 mm
- net VCC: track 433.2 -> 428.3 mm
- net GND: track 718.1 -> 715.6 mm
- net RESET: track 107.6 -> 105.7 mm
- net X-MAX: track 43.9 -> 42.1 mm
- net Y-MAX: track 37.7 -> 36.2 mm
Other:
- outline, holes or cut-outs redrawn
