File: Polarshield v2.1.sch (EAGLE design)
At the start: 82 parts, among them CN1 1X4-CLEANBIG, CN2 1X4-CLEANBIG, CN3 1X4-CLEANBIG, CN4 1X4-CLEANBIG, CN5 1X4-CLEANBIG, CN6 1X4-CLEANBIG, IC1 MP2307, IC2 74541PW, IC3 74541PW, IC4 74541PW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

Commit message: Ran the DRU, ready for making.
Parts:
- removed CN5, CN6: 1X4-CLEANBIG, Polarshield v2.0e:1X4-CLEANBIG
- added JP4, JP5, JP6, JP7: (no value), SparkFun-Connectors:M02POGO_PIN_HOLES_ONLY
- JP1, JP3: device SparkFun-Connectors:M021X02_NO_SILK -> SparkFun-Connectors:M02POGO_PIN_HOLES_ONLY
- JP2: device SparkFun-Connectors:M031X03_NO_SILK -> SparkFun-Connectors:M03POGO_PIN_HOLES_ONLY
Connections:
- net D42: now also JP4.2; no longer CN5.4
- net D43: now also JP4.1; no longer CN6.4
- net D44: now also JP5.2; no longer CN5.3
- net D45: now also JP5.1; no longer CN6.3
- net D46: now also JP6.2; no longer CN5.2
- net D47: now also JP6.1; no longer CN6.2
- net D48: now also JP7.2; no longer CN5.1
- net D49: now also JP7.1; no longer CN6.1

Commit message: v2.1
Parts:
- removed JP15: (no value), pinhead:PINHD-2X3
- added X-MAX, X-MIN, Y-MAX, Y-MIN: (no value), ultimachine:3PIN-HEADER
Connections:
- net GND: now also X-MAX.1, X-MIN.1, Y-MAX.1, Y-MIN.1; no longer JP15.6
- net VCC: now also X-MAX.2, X-MIN.2, Y-MAX.2, Y-MIN.2; no longer JP15.5
- net X-MAX: now also X-MAX.3; no longer JP15.3
- net X-MIN: now also X-MIN.3; no longer JP15.1
- net Y-MAX: now also Y-MAX.3; no longer JP15.4
- net Y-MIN: now also Y-MIN.3; no longer JP15.2
Other:
- note removed: "AUX-1"
- note removed: "AUX-2"
- note removed: "AUX-3"
- note removed: "I2C"
- moved on the sheet: A-MOT1, A-MOT2, A_STP, C1, C14, IC2, IC2P, IC3, IC3P, IC4, IC4P, IC5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
