File: Polarshield v2.5.sch (EAGLE design)
At the start: 83 parts, among them CN1 1X4-CLEANBIG, CN2 1X4-CLEANBIG, CN3 1X4-CLEANBIG, CN4 1X4-CLEANBIG, IC1 MP2307, IC2 74541PW, IC3 74541PW, IC4 74541PW, IC5 74541PW, J1 1X2-3.5MM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

Commit message: Made sch more readable
Other:
- note added: "3.3v buffer ICs"
- note added: "5v buffer IC"
- note added: "buffers"
- note added: "v2.5"
- note removed: "v2.2"
- moved on the sheet: A-MOT1, A_STP, B-MOT1, B-MOT2, B_STP, C-MOT1, C-MOT2, C1, C10, C11, C12, C13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
